Commit message: xacro that builds diff drive robot with wheels and frames to spec

File: nuturtle_description/urdf/diff_drive.urdf.xacro (robot description, xacro)
@@ -7,21 +7,62 @@
 	<xacro:property name="length" value= "${load_yaml('$(find nuturtle_description)/config/diff_params.yaml')['chassis']['length']}"/>
 	<xacro:property name="thickness" value= "${load_yaml('$(find nuturtle_description)/config/diff_params.yaml')['chassis']['thickness']}"/>
+	<!-- macro for making  base_link link -->
 	<xacro:macro name="base_link_gen" params="width length height">
 		<link name="base_link">
 			<visual>
 				<geometry>
-					<box size="${width} ${length} ${height}"/>
+					<box size="${length} ${width} ${height}"/>
 				</geometry>
 				<material name="red_guy">
-					<color rgba="1 0 0 1"/>
+					<color rgba="1 0 0 .5"/>
 				</material>
 			</visual>
 			<collision>
 				<geometry>
-					<box size="${width} ${length} ${height}"/>
+					<box size="${length} ${width} ${height}"/>
 				</geometry>
 			</collision>
 		</link>
 	</xacro:macro>
+	<!-- macro for making wheel links -->
+	<xacro:macro name="wheel_gen" params="name radius width">
+		<link name="${name}">
+			<visual>
+				<geometry>
+					<cylinder radius="${radius}" length="${width}"/>
+				</geometry>
+				<material name="blue_guy">
+					<color rgba="0 0 1 .75"/>
+				</material>
+			</visual>
+			<collision>
+				<geometry>
+					<cylinder radius="${radius}" length="${width}"/>
+				</geometry>
+			</collision>
+		</link>
+	</xacro:macro>
+	<!-- macro for making joints -->
+	<xacro:macro name="joint_gen" params="name parent child origin rotate">
+		<joint name="${name}" type="continuous">
+			<axis xyz="0 0 1"/>
+			<parent link="${parent}"/>
+			<child link="${child}"/>
+			<origin xyz="${-length/4} ${origin}  0" rpy="${pi/2} 0 ${rotate}"/>
+		</joint>
+	</xacro:macro>
+	<!-- generate needed links -->
+	<link name="origin">
+	</link>
 	<xacro:base_link_gen width="${base - width}" length="${length}" height="${thickness}"/>
+	<xacro:wheel_gen radius="${radius}" name="wheel1" width="${width}"/>
+	<xacro:wheel_gen radius="${radius}" name="wheel2" width="${width}"/>
+	<!-- generate joints between links -->
+	<joint name="to_base" type="fixed">
+		<parent link="origin"/>
+		<child link="base_link"/>
+		<origin xyz="0 0 ${radius}" rpy="0 0 ${pi/2}"/>
+	</joint>
+	<xacro:joint_gen name="wheel1_joint" parent="base_link" child="wheel1" origin="${base/2}" rotate="0"/>
+	<xacro:joint_gen name="wheel2_joint" parent="base_link" child="wheel2" origin="${-base/2}" rotate="0"/>
 </robot>

Commit message: finished part A.002 to specifications

File: nuturtle_description/urdf/diff_drive.urdf.xacro (robot description, xacro)
@@ -11,12 +11,14 @@
 		<link name="base_link">
 			<visual>
+				<origin xyz="${length/2 - radius} 0 0" rpy="0 0 0"/>
 				<geometry>
 					<box size="${length} ${width} ${height}"/>
 				</geometry>
 				<material name="red_guy">
-					<color rgba="1 0 0 .5"/>
+					<color rgba="1 0 0 .75"/>
 				</material>
 			</visual>
 			<collision>
+				<origin xyz="${length/2 - radius} 0 0" rpy="0 0 0"/>
 				<geometry>
 					<box size="${length} ${width} ${height}"/>
@@ -29,4 +31,5 @@
 		<link name="${name}">
 			<visual>
+				<origin xyz = "0 0 0" rpy="${pi/2} 0 0"/>
 				<geometry>
 					<cylinder radius="${radius}" length="${width}"/>
@@ -37,6 +40,25 @@
 			</visual>
 			<collision>
+				<origin xyz = "0 0 0" rpy="${pi/2} 0 0"/>
 				<geometry>
 					<cylinder radius="${radius}" length="${width}"/>
+				</geometry>
+			</collision>
+		</link>
+	</xacro:macro>
+	<!-- macro for making caster -->
+	<xacro:macro name="caster_gen" params="name radius">
+		<link name="${name}">
+			<visual>
+				<geometry>
+					<sphere radius="${radius}"/>
+				</geometry>
+				<material name="purp_guy">
+					<color rgba="1 0 1 .5"/>
+				</material>
+			</visual>
+			<collision>
+				<geometry>
+					<sphere radius="${radius}"/>
 				</geometry>
 			</collision>
@@ -46,8 +68,16 @@
 	<xacro:macro name="joint_gen" params="name parent child origin rotate">
 		<joint name="${name}" type="continuous">
-			<axis xyz="0 0 1"/>
+			<axis xyz="0 1 0"/>
 			<parent link="${parent}"/>
 			<child link="${child}"/>
-			<origin xyz="${-length/4} ${origin}  0" rpy="${pi/2} 0 ${rotate}"/>
+			<origin xyz="0 ${origin}  0" rpy="0 0 ${rotate}"/>
+		</joint>
+	</xacro:macro>
+	<!-- macro for caster joints -->
+	<xacro:macro name="caster_joint" params="name parent child origin_z">
+		<joint name="${name}" type="fixed">
+			<parent link="${parent}"/>
+			<child link="${child}"/>
+			<origin xyz="${length/2} 0 ${origin_z}" rpy="0 0 0"/>
 		</joint>
 	</xacro:macro>
@@ -58,4 +88,6 @@
 	<xacro:wheel_gen radius="${radius}" name="wheel1" width="${width}"/>
 	<xacro:wheel_gen radius="${radius}" name="wheel2" width="${width}"/>
+	<xacro:caster_gen radius="${radius/2}" name="caster1"/>
+	<xacro:caster_gen radius="${radius/2}" name="caster2"/>
 	<!-- generate joints between links -->
 	<joint name="to_base" type="fixed">
@@ -64,5 +96,7 @@
 		<origin xyz="0 0 ${radius}" rpy="0 0 ${pi/2}"/>
 	</joint>
-	<xacro:joint_gen name="wheel1_joint" parent="base_link" child="wheel1" origin="${base/2}" rotate="0"/>
-	<xacro:joint_gen name="wheel2_joint" parent="base_link" child="wheel2" origin="${-base/2}" rotate="0"/>
+	<xacro:joint_gen name="left_wheel_axel" parent="base_link" child="wheel1" origin="${base/2}" rotate="0"/>
+	<xacro:joint_gen name="right_wheel_axel" parent="base_link" child="wheel2" origin="${-base/2}" rotate="0"/>
+	<xacro:caster_joint name="cast_joint1" parent="base_link" child="caster1" origin_z="${radius/2}"/>
+	<xacro:caster_joint name="cast_joint2" parent="base_link" child="caster2" origin_z="${-radius/2}"/>
 </robot>

Commit message: removed silly origin link

File: nuturtle_description/urdf/diff_drive.urdf.xacro (robot description, xacro)
@@ -82,7 +82,4 @@
 		</joint>
 	</xacro:macro>
-	<!-- generate needed links -->
-	<link name="origin">
-	</link>
 	<xacro:base_link_gen width="${base - width}" length="${length}" height="${thickness}"/>
 	<xacro:wheel_gen radius="${radius}" name="left_wheel" width="${width}"/>
@@ -90,10 +87,4 @@
 	<xacro:caster_gen radius="${radius/2}" name="caster1"/>
 	<xacro:caster_gen radius="${radius/2}" name="caster2"/>
-	<!-- generate joints between links -->
-	<joint name="to_base" type="fixed">
-		<parent link="origin"/>
-		<child link="base_link"/>
-		<origin xyz="0 0 ${radius}" rpy="0 0 ${pi/2}"/>
-	</joint>
 	<xacro:joint_gen name="left_wheel_axel" parent="base_link" child="left_wheel" origin="${base/2}" rotate="0"/>
 	<xacro:joint_gen name="right_wheel_axel" parent="base_link" child="right_wheel" origin="${-base/2}" rotate="0"/>

Commit message: updated xacro to more accurately resemble turtlebot

File: nuturtle_description/urdf/diff_drive.urdf.xacro (robot description, xacro)
@@ -7,4 +7,5 @@
 	<xacro:property name="length" value= "${load_yaml('$(find nuturtle_description)/config/diff_params.yaml')['chassis']['length']}"/>
 	<xacro:property name="thickness" value= "${load_yaml('$(find nuturtle_description)/config/diff_params.yaml')['chassis']['thickness']}"/>
+	<xacro:property name="height" value= "${load_yaml('$(find nuturtle_description)/config/diff_params.yaml')['chassis']['height']}"/>
 	<!-- macro for making  base_link link -->
 	<xacro:macro name="base_link_gen" params="width length height">
@@ -71,5 +72,5 @@
 			<parent link="${parent}"/>
 			<child link="${child}"/>
-			<origin xyz="0 ${origin}  0" rpy="0 0 ${rotate}"/>
+			<origin xyz="0 ${origin}  ${-height/2}" rpy="0 0 ${rotate}"/>
 		</joint>
 	</xacro:macro>
@@ -79,15 +80,15 @@
 			<parent link="${parent}"/>
 			<child link="${child}"/>
-			<origin xyz="${length/2} 0 ${origin_z}" rpy="0 0 0"/>
+			<origin xyz="${length/2} 0 ${-height/2 - origin_z}" rpy="0 0 0"/>
 		</joint>
 	</xacro:macro>
-	<xacro:base_link_gen width="${base - width}" length="${length}" height="${thickness}"/>
+	<xacro:base_link_gen width="${base - width}" length="${length}" height="${height}"/>
 	<xacro:wheel_gen radius="${radius}" name="left_wheel" width="${width}"/>
 	<xacro:wheel_gen radius="${radius}" name="right_wheel" width="${width}"/>
 	<xacro:caster_gen radius="${radius/2}" name="caster1"/>
-	<xacro:caster_gen radius="${radius/2}" name="caster2"/>
+	<!-- <xacro:caster_gen radius="${radius/2}" name="caster2"/> -->
 	<xacro:joint_gen name="left_wheel_axel" parent="base_link" child="left_wheel" origin="${base/2}" rotate="0"/>
 	<xacro:joint_gen name="right_wheel_axel" parent="base_link" child="right_wheel" origin="${-base/2}" rotate="0"/>
 	<xacro:caster_joint name="cast_joint1" parent="base_link" child="caster1" origin_z="${radius/2}"/>
-	<xacro:caster_joint name="cast_joint2" parent="base_link" child="caster2" origin_z="${-radius/2}"/>
+	<!-- <xacro:caster_joint name="cast_joint2" parent="base_link" child="caster2" origin_z="${-radius/2}"/> -->
 </robot>

Commit message: updated turtlebot urdf and parameters pertaining to it

File: nuturtle_description/urdf/diff_drive.urdf.xacro (robot description, xacro)
@@ -8,4 +8,5 @@
 	<xacro:property name="thickness" value= "${load_yaml('$(find nuturtle_description)/config/diff_params.yaml')['chassis']['thickness']}"/>
 	<xacro:property name="height" value= "${load_yaml('$(find nuturtle_description)/config/diff_params.yaml')['chassis']['height']}"/>
+	<xacro:property name="wheel_axel_offset" value= "${load_yaml('$(find nuturtle_description)/config/diff_params.yaml')['chassis']['wheel_axel_offset']}"/>
 	<!-- macro for making  base_link link -->
 	<xacro:macro name="base_link_gen" params="width length height">
@@ -26,4 +27,22 @@
 				</geometry>
 			</collision>
+			<inertia>
+				<mass value="0.9"/>
+				<inertia ixx="${0.9 * 1.0/12.0 * (width * width + height * height)}" ixy="0.0" ixz="0.0" iyy="${0.9 * 1.0/12.0 * (length * length + height * height)}" iyz="0.0" izz="${0.9 * 1.0/12.0 * (length * length + width * width)}"/>
+			</inertia>
+		</link>
+	</xacro:macro>
+	<!-- macro for making lidar link -->
+	<xacro:macro name="scan_gen" params="radius height">
+		<link name="base_scan">
+			<visual>
+				<origin xyz="0 0 ${height/2}" rpy="0 0 0"/>
+				<geometry>
+					<cylinder radius="${radius}" length="${height}"/>
+				</geometry>
+				<material name="purp_guy">
+					<color rgba="1 0 1 .75"/>
+				</material>
+			</visual>
 		</link>
 	</xacro:macro>
@@ -46,4 +65,8 @@
 				</geometry>
 			</collision>
+			<inertia>
+				<mass value="0.03"/>
+				<inertia ixx="${0.03 * 1.0/12.0 * (3.0 * radius * radius + width * width)}" ixy="0.0" ixz="0.0" iyy="${0.03 * 1.0/12.0 * (3.0 * radius * radius + width * width)}" iyz="0.0" izz="${1.0/2.0 * 0.03 * radius * radius}"/>
+			</inertia>
 		</link>
 	</xacro:macro>
@@ -72,5 +95,5 @@
 			<parent link="${parent}"/>
 			<child link="${child}"/>
-			<origin xyz="0 ${origin}  ${-height/2}" rpy="0 0 ${rotate}"/>
+			<origin xyz="0 ${origin}  ${-height/2 + wheel_axel_offset}" rpy="0 0 ${rotate}"/>
 		</joint>
 	</xacro:macro>
@@ -80,5 +103,13 @@
 			<parent link="${parent}"/>
 			<child link="${child}"/>
-			<origin xyz="${length/2} 0 ${-height/2 - origin_z}" rpy="0 0 0"/>
+			<origin xyz="${length/2} 0 ${-height/2 - origin_z + wheel_axel_offset}" rpy="0 0 0"/>
+		</joint>
+	</xacro:macro>
+	<!-- macro for base_scan joint -->
+	<xacro:macro name="scan_joint" params="name parent child">
+		<joint name="${name}" type="continuous">
+			<parent link="${parent}"/>
+			<child link="${child}"/>
+			<origin xyz="${-radius + length/2} 0 ${height/2}" rpy="0 0 0"/>
 		</joint>
 	</xacro:macro>
@@ -87,8 +118,8 @@
 	<xacro:wheel_gen radius="${radius}" name="right_wheel" width="${width}"/>
 	<xacro:caster_gen radius="${radius/2}" name="caster1"/>
-	<!-- <xacro:caster_gen radius="${radius/2}" name="caster2"/> -->
+	<xacro:scan_gen radius=".03" height=".01"/>
 	<xacro:joint_gen name="left_wheel_axel" parent="base_link" child="left_wheel" origin="${base/2}" rotate="0"/>
 	<xacro:joint_gen name="right_wheel_axel" parent="base_link" child="right_wheel" origin="${-base/2}" rotate="0"/>
 	<xacro:caster_joint name="cast_joint1" parent="base_link" child="caster1" origin_z="${radius/2}"/>
-	<!-- <xacro:caster_joint name="cast_joint2" parent="base_link" child="caster2" origin_z="${-radius/2}"/> -->
+	<xacro:scan_joint name="scan_joint" parent="base_link" child="base_scan"/>
 </robot>

Commit message: added inertial frames to links so they could be erndered and modeled in gazebo

File: nuturtle_description/urdf/diff_drive.urdf.xacro (robot description, xacro)
@@ -1,4 +1,4 @@
 <?xml version="1.0"?>
-<robot xmlns:xacro="http://www.ros.org/wiki/xacro" name="ddiff_drive">
+<robot xmlns:xacro="http://www.ros.org/wiki/xacro" name="nuturtlebot">
 	<!-- load parameters from yaml -->
 	<xacro:property name="width" value= "${load_yaml('$(find nuturtle_description)/config/diff_params.yaml')['wheel']['width']}"/>
@@ -27,8 +27,9 @@
 				</geometry>
 			</collision>
-			<inertia>
+			<inertial>
+				<origin xyz="${length/2 - radius} 0 0" rpy="0 0 0"/>
 				<mass value="0.9"/>
 				<inertia ixx="${0.9 * 1.0/12.0 * (width * width + height * height)}" ixy="0.0" ixz="0.0" iyy="${0.9 * 1.0/12.0 * (length * length + height * height)}" iyz="0.0" izz="${0.9 * 1.0/12.0 * (length * length + width * width)}"/>
-			</inertia>
+			</inertial>
 		</link>
 	</xacro:macro>
@@ -65,8 +66,8 @@
 				</geometry>
 			</collision>
-			<inertia>
+			<inertial>
 				<mass value="0.03"/>
-				<inertia ixx="${0.03 * 1.0/12.0 * (3.0 * radius * radius + width * width)}" ixy="0.0" ixz="0.0" iyy="${0.03 * 1.0/12.0 * (3.0 * radius * radius + width * width)}" iyz="0.0" izz="${1.0/2.0 * 0.03 * radius * radius}"/>
-			</inertia>
+				<inertia ixx="${0.03 * 1.0/12.0 * (3.0 * radius * radius + width * width)}" ixy="0.0" ixz="0.0" izz="${0.03 * 1.0/12.0 * (3.0 * radius * radius + width * width)}" iyz="0.0" iyy="${1.0/2.0 * 0.03 * radius * radius}"/>
+			</inertial>
 		</link>
 	</xacro:macro>
@@ -87,4 +88,6 @@
 				</geometry>
 			</collision>
+<!-- 			<inertial>
+			</inertial> -->
 		</link>
 	</xacro:macro>
@@ -118,8 +121,8 @@
 	<xacro:wheel_gen radius="${radius}" name="right_wheel" width="${width}"/>
 	<xacro:caster_gen radius="${radius/2}" name="caster1"/>
-	<xacro:scan_gen radius=".03" height=".01"/>
+	<!-- <xacro:scan_gen radius=".03" height=".01"/> -->
 	<xacro:joint_gen name="left_wheel_axel" parent="base_link" child="left_wheel" origin="${base/2}" rotate="0"/>
 	<xacro:joint_gen name="right_wheel_axel" parent="base_link" child="right_wheel" origin="${-base/2}" rotate="0"/>
 	<xacro:caster_joint name="cast_joint1" parent="base_link" child="caster1" origin_z="${radius/2}"/>
-	<xacro:scan_joint name="scan_joint" parent="base_link" child="base_scan"/>
+	<!-- <xacro:scan_joint name="scan_joint" parent="base_link" child="base_scan"/> -->
 </robot>

Commit message: added in sensor, fixed typo in mass of wheels

File: nuturtle_description/urdf/diff_drive.urdf.xacro (robot description, xacro)
@@ -67,5 +67,5 @@
 			</collision>
 			<inertial>
-				<mass value="0.03"/>
+				<mass value="0.3"/>
 				<inertia ixx="${0.03 * 1.0/12.0 * (3.0 * radius * radius + width * width)}" ixy="0.0" ixz="0.0" izz="${0.03 * 1.0/12.0 * (3.0 * radius * radius + width * width)}" iyz="0.0" iyy="${1.0/2.0 * 0.03 * radius * radius}"/>
 			</inertial>
@@ -121,8 +121,8 @@
 	<xacro:wheel_gen radius="${radius}" name="right_wheel" width="${width}"/>
 	<xacro:caster_gen radius="${radius/2}" name="caster1"/>
-	<!-- <xacro:scan_gen radius=".03" height=".01"/> -->
+	<xacro:scan_gen radius=".03" height=".01"/>
 	<xacro:joint_gen name="left_wheel_axel" parent="base_link" child="left_wheel" origin="${base/2}" rotate="0"/>
 	<xacro:joint_gen name="right_wheel_axel" parent="base_link" child="right_wheel" origin="${-base/2}" rotate="0"/>
 	<xacro:caster_joint name="cast_joint1" parent="base_link" child="caster1" origin_z="${radius/2}"/>
-	<!-- <xacro:scan_joint name="scan_joint" parent="base_link" child="base_scan"/> -->
+	<xacro:scan_joint name="scan_joint" parent="base_link" child="base_scan"/>
 </robot>

Commit message: added dummy frame for gazebo integration

File: nuturtle_description/urdf/diff_drive.urdf.xacro (robot description, xacro)
@@ -92,4 +92,8 @@
 		</link>
 	</xacro:macro>
+	<xacro:macro name="floor_link">
+		<link name="floor">
+		</link>
+	</xacro:macro>
 	<!-- macro for making joints -->
 	<xacro:macro name="joint_gen" params="name parent child origin rotate">
@@ -111,5 +115,5 @@
 	<!-- macro for base_scan joint -->
 	<xacro:macro name="scan_joint" params="name parent child">
-		<joint name="${name}" type="continuous">
+		<joint name="${name}" type="fixed"> <!-- see if that fixes tf error -->
 			<parent link="${parent}"/>
 			<child link="${child}"/>
@@ -117,4 +121,12 @@
 		</joint>
 	</xacro:macro>
+	<!-- base to floor -->
+	<xacro:macro name="base_to_floor">
+		<joint name="base_to_floor" type="fixed">
+			<parent link="floor"/>
+			<child link="base_link"/>
+		</joint>
+	</xacro:macro>
+	<xacro:floor_link/>
 	<xacro:base_link_gen width="${base - width}" length="${length}" height="${height}"/>
 	<xacro:wheel_gen radius="${radius}" name="left_wheel" width="${width}"/>
@@ -122,4 +134,5 @@
 	<xacro:caster_gen radius="${radius/2}" name="caster1"/>
 	<xacro:scan_gen radius=".03" height=".01"/>
+	<xacro:base_to_floor/>
 	<xacro:joint_gen name="left_wheel_axel" parent="base_link" child="left_wheel" origin="${base/2}" rotate="0"/>
 	<xacro:joint_gen name="right_wheel_axel" parent="base_link" child="right_wheel" origin="${-base/2}" rotate="0"/>
