Commit message: now passing key parameters to pluggin

File: nuturtle_gazebo/urdf/diff_drive.gazebo.xacro (robot description, xacro)
@@ -39,12 +39,13 @@
 		<preserveFixedJoint>true</preserveFixedJoint>
 	</gazebo>
+	<xacro:property name="freq" value= "${load_yaml('$(find nuturtle_description)/config/diff_params.yaml')['freq']}"/>
 	<gazebo>
 	    <plugin name="turtle_drive_plugin" filename="libturtle_drive_plugin.so">
 	      <!-- if joint names not specified, print fatal error and return from Load -->
-	      <left_wheel_joint></left_wheel_joint>
-	      <right_wheel_joint></right_wheel_joint>
-	      <sensor_frequency>200</sensor_frequency> <!-- if not specified should default to 200Hz -->
-	      <wheel_cmd_topic>name_of_wheel_cmd_topic</wheel_cmd_topic>
-	      <sensor_data_topic>name_of_sensor_topic</sensor_data_topic>
+	      <left_wheel_joint>left_wheel_axel</left_wheel_joint>
+	      <right_wheel_joint>right_wheel_axel</right_wheel_joint>
+	      <sensor_frequency>200</sensor_frequency> <!-- if not specified should default to 200Hz "${freq}" -->
+	      <wheel_cmd_topic>wheel_cmd</wheel_cmd_topic>
+	      <sensor_data_topic>sensor_data</sensor_data_topic>
 	    </plugin>
   	</gazebo>

Commit message: added laser scanner to gazebo sdf

File: nuturtle_gazebo/urdf/diff_drive.gazebo.xacro (robot description, xacro)
@@ -50,3 +50,35 @@
 	    </plugin>
   	</gazebo>
+	<gazebo reference="base_scan">
+	  <material>Gazebo/FlatBlack</material>
+	  <sensor type="ray" name="lds_lfcd_sensor">
+	    <pose>0 0 0 0 0 0</pose>
+	    <visualize>true</visualize>
+	    <update_rate>5</update_rate>
+	    <ray>
+	      <scan>
+	        <horizontal>
+	          <samples>360</samples>
+	          <resolution>1</resolution>
+	          <min_angle>0.0</min_angle>
+	          <max_angle>6.28319</max_angle>
+	        </horizontal>
+	      </scan>
+	      <range>
+	        <min>0.120</min>
+	        <max>3.5</max>
+	        <resolution>0.015</resolution>
+	      </range>
+	      <noise>
+	        <type>gaussian</type>
+	        <mean>0.0</mean>
+	        <stddev>0.01</stddev>
+	      </noise>
+	    </ray>
+	    <plugin name="gazebo_ros_lds_lfcd_controller" filename="libgazebo_ros_laser.so">
+	      <topicName>scan</topicName>
+	      <frameName>base_scan</frameName>
+	    </plugin>
+	  </sensor>
+	</gazebo>
 </robot>
